File: sub_schematics/MCIO.kicad_sch (KiCad schematic)
At the start: 1 part

Commit message: Reskew changed skematics
Connections:
- net PCI.RX0+: now also MCIO1.A2 (PER0+); no longer MCIO1.A3 (PER0+)
- net PCI.RX0-: now also MCIO1.A3 (PER0-); no longer MCIO1.A2 (PER0+)
- net PCI.RX1+: now also MCIO1.A5 (PER1+); no longer MCIO1.A6 (PER1-)
- net PCI.RX1-: now also MCIO1.A6 (PER1-); no longer MCIO1.A5 (PER1+)
- net PCI.RX2+: now also MCIO1.A14 (PER2+); no longer MCIO1.A15 (PER2-)
- net PCI.RX2-: now also MCIO1.A15 (PER2-); no longer MCIO1.A14 (PER2+)
- net PCI.RX3+: now also MCIO1.A17 (PER3+); no longer MCIO1.A18 (PER3-)
- net PCI.RX3-: now also MCIO1.A18 (PER3-); no longer MCIO1.A17 (PER3+)
- net PCI.RX4+: now also MCIO1.A20 (PER4+); no longer MCIO1.A21 (PER4-)
- net PCI.RX4-: now also MCIO1.A21 (PER4-); no longer MCIO1.A20 (PER4+)
- net PCI.RX5+: now also MCIO1.A23 (PER5+); no longer MCIO1.A24 (PER5-)
- net PCI.RX5-: now also MCIO1.A24 (PER5-); no longer MCIO1.A23 (PER5+)
- net PCI.RX6+: now also MCIO1.A32 (PER6+); no longer MCIO1.A33 (PER6-)
- net PCI.RX6-: now also MCIO1.A33 (PER6-); no longer MCIO1.A32 (PER6+)
- net PCI.RX7+: now also MCIO1.A35 (PER7+); no longer MCIO1.A36 (PER7+)
- net PCI.RX7-: now also MCIO1.A36 (PER7-); no longer MCIO1.A35 (PER7+)
- net PCI.TX0+: now also MCIO1.B2 (PET0+); no longer MCIO1.B3 (PET0-)
- net PCI.TX0-: now also MCIO1.B3 (PET0-); no longer MCIO1.B2 (PET0+)
- net PCI.TX1+: now also MCIO1.B5 (PET1+); no longer MCIO1.B6 (PET1-)
- net PCI.TX1-: now also MCIO1.B6 (PET1-); no longer MCIO1.B5 (PET1+)
- net PCI.TX2+: now also MCIO1.B14 (PET2+); no longer MCIO1.B15 (PET2-)
- net PCI.TX2-: now also MCIO1.B15 (PET2-); no longer MCIO1.B14 (PET2+)
- net PCI.TX3+: now also MCIO1.B17 (PET3+); no longer MCIO1.B18 (PET3-)
- net PCI.TX3-: now also MCIO1.B18 (PET3-); no longer MCIO1.B17 (PET3+)
- net PCI.TX4+: now also MCIO1.B20 (PET4+); no longer MCIO1.B21 (PET4-)
- net PCI.TX4-: now also MCIO1.B21 (PET4-); no longer MCIO1.B20 (PET4+)
- net PCI.TX5+: now also MCIO1.B23 (PET5+); no longer MCIO1.B24 (PET5-)
- net PCI.TX5-: now also MCIO1.B24 (PET5-); no longer MCIO1.B23 (PET5+)
- net PCI.TX6+: now also MCIO1.B32 (PET6+); no longer MCIO1.B33 (PET6-)
- net PCI.TX6-: now also MCIO1.B33 (PET6-); no longer MCIO1.B32 (PET6+)
- net PCI.TX7+: now also MCIO1.B35 (PET7+); no longer MCIO1.B36 (PET7-)
- net PCI.TX7-: now also MCIO1.B36 (PET7-); no longer MCIO1.B35 (PET7+)
Changed lines of the file:
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@@
 		)
 	)
-	(label "PCI.TX5+"
+	(label "PCI.RX2+"
+		(at 46.99 68.58 0)
+		(effects
+			(font
+				(size 1.27 1.27)
+			)
+			(justify left bottom)
+		)
+	)
+	(label "PCI.TX5-"
 		(at 113.03 93.98 180)
 		(effects
@@
 		)
 	)
-	(label "PCI.TX6+"
+	(label "PCI.TX6-"
 		(at 113.03 116.84 180)
 		(effects
@@
 		)
 	)
-	(label "PCI.RX6+"
+	(label "PCI.RX0+"
+		(at 46.99 38.1 0)
+		(effects
+			(font
+				(size 1.27 1.27)
+			)
+			(justify left bottom)
+		)
+	)
+	(label "PCI.RX6-"
 		(at 46.99 116.84 0)
 		(effects
@@
 		)
 	)
-	(label "PCI.TX4-"
+	(label "PCI.TX4+"
 		(at 113.03 83.82 180)
 		(effects
@@
 		)
 	)
-	(label "PCI.TX0+"
+	(label "PCI.RX1+"
+		(at 46.99 45.72 0)
+		(effects
+			(font
+				(size 1.27 1.27)
+			)
+			(justify left bottom)
+		)
+	)
+	(label "PCI.TX0-"
 		(at 113.03 40.64 180)
 		(effects
@@
 		)
 	)
-	(label "PCI.RX6-"
+	(label "PCI.RX6+"
 		(at 46.99 114.3 0)
 		(effects
@@
 		)
 	)
-	(label "PCI.TX6-"
+	(label "PCI.TX6+"
 		(at 113.03 114.3 180)
 		(effects
@@
 		)
 	)
+	(label "PCI.TX7-"
+		(at 113.03 124.46 180)
+		(effects
+			(font
+				(size 1.27 1.27)
+			)
+			(justify right bottom)
+		)
+	)
+	(label "PCI.RX0-"
+		(at 46.99 40.64 0)
+		(effects
+			(font
+				(size 1.27 1.27)
+			)
+			(justify left bottom)
+		)
+	)
+	(label "PCI.TX2-"
+		(at 113.03 71.12 180)
+		(effects
+			(font
+				(size 1.27 1.27)
+			)
+			(justify right bottom)
+		)
+	)
+	(label "PCI.RX2-"
+		(at 46.99 71.12 0)
+		(effects
+			(font
+				(size 1.27 1.27)
+			)
+			(justify left bottom)
+		)
+	)
+	(label "PCI.TX1-"
+		(at 113.03 48.26 180)
+		(effects
+			(font
+				(size 1.27 1.27)
+			)
+			(justify right bottom)
+		)
+	)
+	(label "PCI.RX7-"
+		(at 46.99 124.46 0)
+		(effects
+			(font
+				(size 1.27 1.27)
+			)
+			(justify left bottom)
+		)
+	)
+	(label "PCI.RX5+"
+		(at 46.99 91.44 0)
+		(effects
+			(font
+				(size 1.27 1.27)
+			)
+			(justify left bottom)
+		)
+	)
+	(label "PCI.RX4-"
+		(at 46.99 86.36 0)
+		(effects
+			(font
+				(size 1.27 1.27)
+			)
+			(justify left bottom)
+		)
+	)
+	(label "PCI.TX3-"
+		(at 113.03 78.74 180)
+		(effects
+			(font
+				(size 1.27 1.27)
+			)
+			(justify right bottom)
+		)
+	)
+	(label "PCI.RX4+"
+		(at 46.99 83.82 0)
+		(effects
+			(font
+				(size 1.27 1.27)
+			)
+			(justify left bottom)
+		)
+	)
+	(label "PCI.TX3+"
+		(at 113.03 76.2 180)
+		(effects
+			(font
+				(size 1.27 1.27)
+			)
+			(justify right bottom)
+		)
+	)
 	(label "PCI.TX7+"
-		(at 113.03 124.46 180)
-		(effects
-			(font
-				(size 1.27 1.27)
-			)
-			(justify right bottom)
-		)
-	)
-	(label "PCI.TX2+"
-		(at 113.03 71.12 180)
-		(effects
-			(font
-				(size 1.27 1.27)
-			)
-			(justify right bottom)
-		)
-	)
-	(label "PCI.TX1+"
-		(at 113.03 48.26 180)
-		(effects
-			(font
-				(size 1.27 1.27)
-			)
-			(justify right bottom)
-		)
-	)
-	(label "PCI.RX7+"
-		(at 46.99 124.46 0)
-		(effects
-			(font
-				(size 1.27 1.27)
-			)
-			(justify left bottom)
-		)
-	)
-	(label "PCI.RX5-"
-		(at 46.99 91.44 0)
-		(effects
-			(font
-				(size 1.27 1.27)
-			)
-			(justify left bottom)
-		)
-	)
-	(label "PCI.RX4+"
-		(at 46.99 86.36 0)
-		(effects
-			(font
-				(size 1.27 1.27)
-			)
-			(justify left bottom)
-		)
-	)
-	(label "PCI.TX3+"
-		(at 113.03 78.74 180)
-		(effects
-			(font
-				(size 1.27 1.27)
-			)
-			(justify right bottom)
-		)
-	)
-	(label "PCI.RX2+"
-		(at 46.99 71.12 0)
-		(effects
-			(font
-				(size 1.27 1.27)
-			)
-			(justify left bottom)
-		)
-	)
-	(label "PCI.RX4-"
-		(at 46.99 83.82 0)
-		(effects
-			(font
-				(size 1.27 1.27)
-			)
-			(justify left bottom)
-		)
-	)
-	(label "PCI.TX3-"
-		(at 113.03 76.2 180)
-		(effects
-			(font
-				(size 1.27 1.27)
-			)
-			(justify right bottom)
-		)
-	)
-	(label "PCI.RX0+"
-		(at 46.99 40.64 0)
-		(effects
-			(font
-				(size 1.27 1.27)
-			)
-			(justify left bottom)
-		)
-	)
-	(label "PCI.RX1+"
-		(at 46.99 48.26 0)
-		(effects
-			(font
-				(size 1.27 1.27)
-			)
-			(justify left bottom)
-		)
-	)
-	(label "PCI.RX0-"
-		(at 46.99 38.1 0)
-		(effects
-			(font
-				(size 1.27 1.27)
-			)
-			(justify left bottom)
-		)
-	)
-	(label "PCI.TX7-"
 		(at 113.03 121.92 180)
 		(effects
@@
 		)
 	)
-	(label "PCI.TX5-"
+	(label "PCI.TX5+"
 		(at 113.03 91.44 180)
+		(effects
+			(font
+				(size 1.27 1.27)
+			)
+			(justify right bottom)
+		)
+	)
+	(label "PCI.TX0+"
+		(at 113.03 38.1 180)
+		(effects
+			(font
+				(size 1.27 1.27)
+			)
+			(justify right bottom)
+		)
+	)
+	(label "PCI.TX4-"
+		(at 113.03 86.36 180)
+		(effects
+			(font
+				(size 1.27 1.27)
+			)
+			(justify right bottom)
+		)
+	)
+	(label "PCI.RX5-"
+		(at 46.99 93.98 0)
+		(effects
+			(font
+				(size 1.27 1.27)
+			)
+			(justify left bottom)
+		)
+	)
+	(label "PEX.SDA"
+		(at 102.87 55.88 0)
+		(effects
+			(font
+				(size 1.27 1.27)
+			)
+			(justify left bottom)
+		)
+	)
+	(label "PCI.RX3+"
+		(at 46.99 76.2 0)
+		(effects
+			(font
+				(size 1.27 1.27)
+			)
+			(justify left bottom)
+		)
+	)
+	(label "PCI.TX1+"
+		(at 113.03 45.72 180)
 		(effects
 			(font
@@
 		)
 	)
-	(label "PCI.TX0-"
-		(at 113.03 38.1 180)
-		(effects
-			(font
-				(size 1.27 1.27)
-			)
-			(justify right bottom)
-		)
-	)
-	(label "PCI.TX4+"
-		(at 113.03 86.36 180)
-		(effects
-			(font
-				(size 1.27 1.27)
-			)
-			(justify right bottom)
-		)
-	)
-	(label "PCI.RX5+"
-		(at 46.99 93.98 0)
+	(label "PCI.TX2+"
+		(at 113.03 68.58 180)
+		(effects
+			(font
+				(size 1.27 1.27)
+			)
+			(justify right bottom)
+		)
+	)
+	(label "PCI.RX7+"
+		(at 46.99 121.92 0)
+		(effects
+			(font
+				(size 1.27 1.27)
+			)
+			(justify left bottom)
+		)
+	)
+	(label "PCI.RX1-"
+		(at 46.99 48.26 0)
 		(effects
 			(font
@@
 	)
 	(label "PCI.RX3-"
-		(at 46.99 76.2 0)
-		(effects
-			(font
-				(size 1.27 1.27)
-			)
-			(justify left bottom)
-		)
-	)
-	(label "PCI.TX1-"
-		(at 113.03 45.72 180)
-		(effects
-			(font
-				(size 1.27 1.27)
-			)
-			(justify right bottom)
-		)
-	)
-	(label "PCI.RX1-"
-		(at 46.99 45.72 0)
-		(effects
-			(font
-				(size 1.27 1.27)
-			)
-			(justify left bottom)
-		)
-	)
-	(label "PEX.SDA"
-		(at 102.87 55.88 0)
-		(effects
-			(font
-				(size 1.27 1.27)
-			)
-			(justify left bottom)
-		)
-	)
-	(label "PCI.TX2-"
-		(at 113.03 68.58 180)
-		(effects
-			(font
-				(size 1.27 1.27)
-			)
-			(justify right bottom)
-		)
-	)
-	(label "PCI.RX7-"
-		(at 46.99 121.92 0)
-		(effects
-			(font
-				(size 1.27 1.27)
-			)
-			(justify left bottom)
-		)
-	)
-	(label "PCI.RX2-"
-		(at 46.99 68.58 0)
-		(effects
-			(font
-				(size 1.27 1.27)
-			)
-			(justify left bottom)
-		)
-	)
-	(label "PCI.RX3+"
 		(at 46.99 78.74 0)
 		(effects
@@
 			)
 		)
-		(property "Datasheet" ""
+		(property "Datasheet" "https://www.amphenol-cs.com/product/g97r22312hr.html"
 			(at 80.01 87.63 0)
 			(hide yes)
