File: sub_schematics/PCIe_retimer.kicad_sch (KiCad schematic)
At the start: 2 parts, among them U1 SY75602ATWL-TR

Commit message: updated kicad oot
Parts:
- U1: footprint pcie-clk-mux:VDFN8_NNC_MCH -> pcie-clk-buffer:VDFN8_NNC_MCH; symbol pcie-clk-mux:SY75602ATWL-TR -> pcie-clk-buffer:SY75602ATWL-TR
Changed lines of the file:
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@@
 	)
 	(symbol
-		(lib_id "pcie-clk-mux:SY75602ATWL-TR")
+		(lib_id "pcie-clk-buffer:SY75602ATWL-TR")
 		(at 184.15 170.18 0)
 		(unit 1)
@@
 		(fields_autoplaced yes)
 		(property "Reference" "U1"
-			(at 184.15 158.75 0)
+			(at 184.15 161.29 0)
 			(show_name no)
 			(do_not_autoplace no)
@@
 		)
 		(property "Value" "SY75602ATWL-TR"
-			(at 184.15 161.29 0)
+			(at 184.15 165.1 0)
+			(hide yes)
 			(show_name no)
 			(do_not_autoplace no)
@@
 			)
 		)
-		(property "Footprint" "pcie-clk-mux:VDFN8_NNC_MCH"
+		(property "Footprint" "pcie-clk-buffer:VDFN8_NNC_MCH"
 			(at 183.896 153.67 0)
 			(hide yes)
@@
 		)
 		(property "JLCPCB Part #" "C3613417"
-			(at 184.15 170.18 0)
+			(at 184.15 156.972 0)
 			(hide yes)
 			(show_name no)
@@
 		)
 		(property "MPN" "SY75602ATWL-TR"
-			(at 184.15 170.18 0)
+			(at 184.15 156.972 0)
 			(hide yes)
 			(show_name no)

Commit message: schematics fixup
Parts:
- removed C3: 0402_885012105020, WE_WCAP-CSGP:C_Wurth_WCAP-CSGP-0402, symbol WE_WCAP-CSGP:0402_885012105020
Connections:
- net PWR.3V3: now also U1.8 (VDD)
